File: data_logger/data_logger.sch (KiCad schematic (older format))
At the start: 7 parts

Commit message: some setup
Parts:
- added D?: LED, symbol Device:LED
- added J?: USB_B_Micro, symbol Connector:USB_B_Micro
- added J?: Micro_SD_Card, symbol Connector:Micro_SD_Card
- added R? (x2): R, symbol Device:R
- added SW?: SW_Push_Open, symbol Switch:SW_Push_Open
- added U?: BD1020HFV, Package_TO_SOT_SMD:HVSOF5, symbol Sensor_Temperature:BD1020HFV
Connections:
- wire segments 30 -> 53
Other:
- note added: "Look up how the USB connector has to be set up"
- note added: "Needs Crystal\n"
- note added: "Needs to be modified so it can\nbe pulled high when programming\n\n"
- note added: "Possible Sensors\nBarometer\nLux\n"
- note added: "Power Indicator"
- note added: "REMEMBER TO CHECK ALL MAXIMUM VOLTAGE RATINGS\n"
- note added: "WiFi/Bluetooth/RF module\n"
Changed lines of the file:
@@
 L Device:R R?
 U 1 1 5B9F2FC0
-P 7300 2300
-F 0 "R?" H 7370 2346 50  0000 L CNN
-F 1 "10K" H 7370 2255 50  0000 L CNN
-F 2 "" V 7230 2300 50  0001 C CNN
-F 3 "~" H 7300 2300 50  0001 C CNN
-	1    7300 2300
-	1    0    0    -1
+P 6650 2200
+F 0 "R?" V 6443 2200 50  0000 C CNN
+F 1 "10K" V 6534 2200 50  0000 C CNN
+F 2 "" V 6580 2200 50  0001 C CNN
+F 3 "~" H 6650 2200 50  0001 C CNN
+	1    6650 2200
+	0    1    1    0
 $EndComp
 $Comp
@@
 Wire Wire Line
 	7150 2600 7300 2600
-Wire Wire Line
-	7300 2600 7300 2450
-Wire Wire Line
-	7300 2600 7300 2750
-Connection ~ 7300 2600
 $Comp
 L power:GND #PWR?
@@
 Wire Wire Line
 	9900 2150 10050 2150
-Text Label 7300 2000 2    50   ~ 0
-VDD
-Wire Wire Line
-	7300 2000 7300 2150
+Text Label 6500 1900 2    50   ~ 0
+VDD
 Wire Wire Line
 	4950 2300 4950 1400
@@
 Wire Wire Line
 	2950 4500 3250 4500
+$Comp
+L Sensor_Temperature:BD1020HFV U?
+U 1 1 5B9F57E0
+P 2100 3100
+F 0 "U?" H 2100 3467 50  0000 C CNN
+F 1 "BD1020HFV" H 2100 3376 50  0000 C CNN
+F 2 "Package_TO_SOT_SMD:HVSOF5" H 2100 2700 50  0001 C CNN
+F 3 "http://rohmfs.rohm.com/en/products/databook/datasheet/ic/sensor/temperature/bd1020hfv-e.pdf" H 2100 3100 50  0001 C CNN
+	1    2100 3100
+	1    0    0    -1
+$EndComp
+Text Label 1550 2700 0    50   ~ 0
+VDD
+Wire Wire Line
+	1550 3000 1700 3000
+Wire Wire Line
+	1550 2700 1550 3000
+$Comp
+L power:GND #PWR?
+U 1 1 5B9F6328
+P 2500 3350
+F 0 "#PWR?" H 2500 3100 50  0001 C CNN
+F 1 "GND" H 2505 3177 50  0000 C CNN
+F 2 "" H 2500 3350 50  0001 C CNN
+F 3 "" H 2500 3350 50  0001 C CNN
+	1    2500 3350
+	1    0    0    -1
+$EndComp
+Wire Wire Line
+	2500 3200 2500 3350
+Wire Wire Line
+	2500 3000 3250 3000
+Wire Wire Line
+	3250 2950 3250 3000
+Connection ~ 3250 3000
+Wire Wire Line
+	1700 3100 1700 3200
+Wire Wire Line
+	1700 3350 2500 3350
+Connection ~ 1700 3200
+Wire Wire Line
+	1700 3200 1700 3350
+Connection ~ 2500 3350
+Text Notes 900  800  0    50   ~ 0
+REMEMBER TO CHECK ALL MAXIMUM VOLTAGE RATINGS\n
+$Comp
+L Connector:USB_B_Micro J?
+U 1 1 5B9F7E9F
+P 2650 5500
+F 0 "J?" H 2705 5967 50  0000 C CNN
+F 1 "USB_B_Micro" H 2705 5876 50  0000 C CNN
+F 2 "" H 2800 5450 50  0001 C CNN
+F 3 "~" H 2800 5450 50  0001 C CNN
+	1    2650 5500
+	1    0    0    -1
+$EndComp
+Wire Wire Line
+	2950 5600 3100 5600
+Wire Wire Line
+	3100 5600 3100 4600
+Wire Wire Line
+	3100 4600 3250 4600
+Wire Wire Line
+	2950 5500 3250 5500
+Wire Wire Line
+	3250 5500 3250 4700
+$Comp
+L Device:LED D?
+U 1 1 5B9F95F6
+P 9850 3550
+F 0 "D?" V 9888 3433 50  0000 R CNN
+F 1 "LED" V 9797 3433 50  0000 R CNN
+F 2 "" H 9850 3550 50  0001 C CNN
+F 3 "~" H 9850 3550 50  0001 C CNN
+	1    9850 3550
+	0    -1   -1   0
+$EndComp
+$Comp
+L Device:R R?
+U 1 1 5B9FA85A
+P 9500 3150
+F 0 "R?" H 9570 3196 50  0000 L CNN
+F 1 "R" H 9570 3105 50  0000 L CNN
+F 2 "" V 9430 3150 50  0001 C CNN
+F 3 "~" H 9500 3150 50  0001 C CNN
+	1    9500 3150
+	1    0    0    -1
+$EndComp
+$Comp
+L Device:R R?
+U 1 1 5B9FA95C
+P 9500 3600
+F 0 "R?" H 9570 3646 50  0000 L CNN
+F 1 "R" H 9570 3555 50  0000 L CNN
+F 2 "" V 9430 3600 50  0001 C CNN
+F 3 "~" H 9500 3600 50  0001 C CNN
+	1    9500 3600
+	1    0    0    -1
+$EndComp
+Text Label 9500 2750 0    50   ~ 0
+VDD
+Wire Wire Line
+	9500 2750 9500 3000
+Wire Wire Line
+	9500 3300 9500 3400
+$Comp
+L power:GND #PWR?
+U 1 1 5B9FBDFD
+P 9500 4000
+F 0 "#PWR?" H 9500 3750 50  0001 C CNN
+F 1 "GND" H 9505 3827 50  0000 C CNN
+F 2 "" H 9500 4000 50  0001 C CNN
+F 3 "" H 9500 4000 50  0001 C CNN
+	1    9500 4000
+	1    0    0    -1
+$EndComp
+Wire Wire Line
+	9500 4050 9500 4000
+Connection ~ 9500 4000
+Wire Wire Line
+	9500 4000 9500 3900
+Wire Wire Line
+	9500 3900 9850 3900
+Wire Wire Line
+	9850 3900 9850 3700
+Connection ~ 9500 3900
+Wire Wire Line
+	9500 3900 9500 3750
+Wire Wire Line
+	9850 3400 9500 3400
+Connection ~ 9500 3400
+Wire Wire Line
+	9500 3400 9500 3450
+Text Notes 9600 2900 0    50   ~ 0
+Power Indicator
+Text Notes 2100 6100 0    50   ~ 0
+Look up how the USB connector has to be set up
+Text Notes 900  1300 0    50   ~ 0
+Possible Sensors\nBarometer\nLux\n
+$Comp
+L Connector:Micro_SD_Card J?
+U 1 1 5B9FE1CF
+P 9900 5250
+F 0 "J?" H 9850 5967 50  0000 C CNN
+F 1 "Micro_SD_Card" H 9850 5876 50  0000 C CNN
+F 2 "" H 11050 5550 50  0001 C CNN
+F 3 "http://katalog.we-online.de/em/datasheet/693072010801.pdf" H 9900 5250 50  0001 C CNN
+	1    9900 5250
+	1    0    0    -1
+$EndComp
+Text Notes 9450 6150 0    50   ~ 0
+Needs Crystal\n
+Text Notes 9350 1000 0    50   ~ 0
+WiFi/Bluetooth/RF module\n
+Text Notes 6650 1850 0    50   ~ 0
+Needs to be modified so it can\nbe pulled high when programming\n\n
+Wire Wire Line
+	7300 2600 7300 2750
+$Comp
+L Switch:SW_Push_Open SW?
+U 1 1 5B9FE51E
+P 7700 2400
+F 0 "SW?" V 7654 2477 50  0000 L CNN
+F 1 "SW_Push_Open" V 7745 2477 50  0000 L CNN
+F 2 "" H 7700 2600 50  0001 C CNN
+F 3 "" H 7700 2600 50  0001 C CNN
+	1    7700 2400
+	0    1    1    0
+$EndComp
+Connection ~ 7300 2600
+Wire Wire Line
+	7300 2600 7700 2600
+Wire Wire Line
+	6800 2200 7700 2200
+Wire Wire Line
+	6500 1900 6500 2200
 $EndSCHEMATC

Commit message: added barometer, photoresistor, and connected micro-usb
Parts:
- added MH?: PRV, symbol Mechanical:MountingHole_Pad
- added MH?: PRG, symbol Mechanical:MountingHole_Pad
- added R?: R, symbol Device:R
- added U?: MS5637, barometer custom, symbol Custom_Symbols:MS5637
Connections:
- net labels added: +5V, SCL, SDA
- wire segments 53 -> 74
Other:
- note added: "Pins for Photoresister\nDiameter still needs modification"
- note removed: "Possible Sensors\nBarometer\nLux\n"
Changed lines of the file:
@@
 EESchema Schematic File Version 4
+LIBS:data_logger-cache
 EELAYER 26 0
 EELAYER END
@@
 U 1 1 5B9F2FC0
 P 6650 2200
-F 0 "R?" V 6443 2200 50  0000 C CNN
+F 0 "R?" V 6450 2200 50  0000 C CNN
 F 1 "10K" V 6534 2200 50  0000 C CNN
 F 2 "" V 6580 2200 50  0001 C CNN
@@
 Text Notes 2100 6100 0    50   ~ 0
 Look up how the USB connector has to be set up
-Text Notes 900  1300 0    50   ~ 0
-Possible Sensors\nBarometer\nLux\n
 $Comp
 L Connector:Micro_SD_Card J?
@@
 Wire Wire Line
 	6500 1900 6500 2200
+$Comp
+L Custom_Symbols:MS5637 U?
+U 1 1 5BA062B8
+P 3150 1400
+F 0 "U?" H 3150 1515 50  0000 C CNN
+F 1 "MS5637" H 3150 1424 50  0000 C CNN
+F 2 "barometer custom" H 3150 1400 50  0001 C CNN
+F 3 "https://www.mouser.com/datasheet/2/418/NG_DS_MS5637-02BA03_B1-1130139.pdf" H 3150 1400 50  0001 C CNN
+	1    3150 1400
+	1    0    0    -1
+$EndComp
+Text Label 3850 1600 0    50   ~ 0
+VDD
+Text Label 6800 3800 0    50   ~ 0
+SDA
+Wire Wire Line
+	6800 3800 6650 3800
+Text Label 6800 3900 0    50   ~ 0
+SCL
+Wire Wire Line
+	6800 3900 6650 3900
+Text Label 2700 1600 2    50   ~ 0
+SDA
+Text Label 2550 1850 0    50   ~ 0
+SCL
+Wire Wire Line
+	3550 1600 3850 1600
+Wire Wire Line
+	2600 1600 2750 1600
+Wire Wire Line
+	2550 1850 2750 1850
+$Comp
+L power:GND #PWR?
+U 1 1 5BA215B2
+P 3850 1850
+F 0 "#PWR?" H 3850 1600 50  0001 C CNN
+F 1 "GND" H 3855 1677 50  0000 C CNN
+F 2 "" H 3850 1850 50  0001 C CNN
+F 3 "" H 3850 1850 50  0001 C CNN
+	1    3850 1850
+	1    0    0    -1
+$EndComp
+Wire Wire Line
+	3850 1850 3550 1850
+$Comp
+L Mechanical:MountingHole_Pad MH?
+U 1 1 5BA25681
+P 1700 4000
+F 0 "MH?" H 2000 4000 50  0000 R CNN
+F 1 "PRV" H 2000 4100 50  0000 R CNN
+F 2 "" H 1700 4000 50  0001 C CNN
+F 3 "~" H 1700 4000 50  0001 C CNN
+	1    1700 4000
+	-1   0    0    1
+$EndComp
+$Comp
+L Mechanical:MountingHole_Pad MH?
+U 1 1 5BA25850
+P 1900 4000
+F 0 "MH?" H 1800 3958 50  0000 R CNN
+F 1 "PRG" H 1800 4050 50  0000 R CNN
+F 2 "" H 1900 4000 50  0001 C CNN
+F 3 "~" H 1900 4000 50  0001 C CNN
+	1    1900 4000
+	-1   0    0    1
+$EndComp
+Text Label 1200 3550 0    50   ~ 0
+VDD
+Wire Wire Line
+	1200 3550 1700 3550
+Wire Wire Line
+	1700 3550 1700 3900
+$Comp
+L Device:R R?
+U 1 1 5BA2875E
+P 2250 3800
+F 0 "R?" H 2320 3846 50  0000 L CNN
+F 1 "R" H 2320 3755 50  0000 L CNN
+F 2 "" V 2180 3800 50  0001 C CNN
+F 3 "~" H 2250 3800 50  0001 C CNN
+	1    2250 3800
+	0    1    1    0
+$EndComp
+Wire Wire Line
+	1900 3900 1900 3800
+Wire Wire Line
+	1900 3800 2100 3800
+$Comp
+L power:GND #PWR?
+U 1 1 5BA3000B
+P 2500 3850
+F 0 "#PWR?" H 2500 3600 50  0001 C CNN
+F 1 "GND" H 2505 3677 50  0000 C CNN
+F 2 "" H 2500 3850 50  0001 C CNN
+F 3 "" H 2500 3850 50  0001 C CNN
+	1    2500 3850
+	1    0    0    -1
+$EndComp
+Wire Wire Line
+	2500 3850 2500 3800
+Wire Wire Line
+	2500 3800 2400 3800
+Wire Wire Line
+	1900 3800 1900 3650
+Wire Wire Line
+	1900 3650 3150 3650
+Wire Wire Line
+	3150 3650 3150 3100
+Wire Wire Line
+	3150 3100 3250 3100
+Connection ~ 1900 3800
+Text Notes 1200 4300 0    50   ~ 0
+Pins for Photoresister\nDiameter still needs modification
+Wire Wire Line
+	2650 5900 4950 5900
+Wire Wire Line
+	4950 5900 4950 5550
+Connection ~ 4950 5550
+$Comp
+L power:+5V #PWR?
+U 1 1 5BA3B6F3
+P 1850 4950
+F 0 "#PWR?" H 1850 4800 50  0001 C CNN
+F 1 "+5V" H 1865 5123 50  0000 C CNN
+F 2 "" H 1850 4950 50  0001 C CNN
+F 3 "" H 1850 4950 50  0001 C CNN
+	1    1850 4950
+	1    0    0    -1
+$EndComp
+Wire Wire Line
+	2950 4950 2950 5300
+Wire Wire Line
+	1850 4950 2950 4950
+Wire Wire Line
+	2550 5900 2650 5900
+Connection ~ 2650 5900
 $EndSCHEMATC

Commit message: Added wifi module
Parts:
- removed J?: Micro_SD_Card, symbol Connector:Micro_SD_Card
- added U?: ESP-WROOM-02, symbol wifi:ESP-WROOM-02
Connections:
- net labels added: RST
- wire segments 74 -> 97
Other:
- note added: "Figure out rest of ports and power for wifi module\n"
- note removed: "Look up how the USB connector has to be set up"
- note removed: "Needs Crystal\n"
- note removed: "WiFi/Bluetooth/RF module\n"

Commit message: forgot to save
Parts:
- gave numbers to parts that had none: 18
Changed lines of the file:
@@
 $EndDescr
 $Comp
-L MCU_Microchip_PIC18:PIC18F45K50_QFP U?
+L MCU_Microchip_PIC18:PIC18F45K50_QFP U3
 U 1 1 5B9F2A46
 P 4950 3700
-F 0 "U?" H 4950 5278 50  0000 C CNN
+F 0 "U3" H 4950 5278 50  0000 C CNN
 F 1 "PIC18F45K50_QFP" H 4950 5187 50  0000 C CNN
 F 2 "Package_QFP:TQFP-44_10x10mm_P0.8mm" H 4950 3700 50  0001 C CIN
@@
 $EndComp
 $Comp
-L Device:C C?
+L Device:C C3
 U 1 1 5B9F2BB1
 P 10400 3650
-F 0 "C?" H 10515 3696 50  0000 L CNN
+F 0 "C3" H 10515 3696 50  0000 L CNN
 F 1 ".uF 20V" H 10515 3605 50  0000 L CNN
 F 2 "" H 10438 3500 50  0001 C CNN
@@
 $EndComp
 $Comp
-L Device:C C?
+L Device:C C4
 U 1 1 5B9F2DE1
 P 10650 3400
-F 0 "C?" H 10765 3446 50  0000 L CNN
+F 0 "C4" H 10765 3446 50  0000 L CNN
 F 1 ".uF 20V" H 10765 3355 50  0000 L CNN
 F 2 "" H 10688 3250 50  0001 C CNN
@@
 $EndComp
 $Comp
-L Device:C C?
+L Device:C C1
 U 1 1 5B9F2F6D
 P 2800 4500
-F 0 "C?" V 2548 4500 50  0000 C CNN
+F 0 "C1" V 2548 4500 50  0000 C CNN
 F 1 ".uF 20V" V 2639 4500 50  0000 C CNN
 F 2 "" H 2838 4350 50  0001 C CNN
@@
 $EndComp
 $Comp
-L Device:C C?
+L Device:C C2
 U 1 1 5B9F2F96
 P 7300 2900
-F 0 "C?" H 7415 2946 50  0000 L CNN
+F 0 "C2" H 7415 2946 50  0000 L CNN
 F 1 ".uF 20V" H 7415 2855 50  0000 L CNN
 F 2 "" H 7338 2750 50  0001 C CNN
@@
 $EndComp
 $Comp
-L Device:R R?
+L Device:R R4
 U 1 1 5B9F2FC0
 P 6350 2200
-F 0 "R?" V 6150 2200 50  0000 C CNN
+F 0 "R4" V 6150 2200 50  0000 C CNN
 F 1 "10K" V 6234 2200 50  0000 C CNN
 F 2 "" V 6280 2200 50  0001 C CNN
@@
 $EndComp
 $Comp
-L Device:R R?
+L Device:R R5
 U 1 1 5B9F32F1
 P 7000 2600
-F 0 "R?" V 7207 2600 50  0000 C CNN
+F 0 "R5" V 7207 2600 50  0000 C CNN
 F 1 "100" V 7116 2600 50  0000 C CNN
 F 2 "" V 6930 2600 50  0001 C CNN
@@
 	7150 2600 7300 2600
 $Comp
-L power:GND #PWR?
+L power:GND #PWR0101
 U 1 1 5B9F342B
 P 7300 3200
-F 0 "#PWR?" H 7300 2950 50  0001 C CNN
+F 0 "#PWR0101" H 7300 2950 50  0001 C CNN
 F 1 "GND" H 7305 3027 50  0000 C CNN
 F 2 "" H 7300 3200 50  0001 C CNN
@@
 	7300 3050 7300 3200
 $Comp
-L power:VDD #PWR?
+L power:VDD #PWR0102
 U 1 1 5B9F3490
 P 1400 7300
-F 0 "#PWR?" H 1400 7150 50  0001 C CNN
+F 0 "#PWR0102" H 1400 7150 50  0001 C CNN
 F 1 "VDD" H 1417 7473 50  0000 C CNN
 F 2 "" H 1400 7300 50  0001 C CNN
@@
 Connection ~ 5050 1500
 $Comp
-L power:GND #PWR?
+L power:GND #PWR0103
 U 1 1 5B9F47C6
 P 5300 5700
-F 0 "#PWR?" H 5300 5450 50  0001 C CNN
+F 0 "#PWR0103" H 5300 5450 50  0001 C CNN
 F 1 "GND" H 5305 5527 50  0000 C CNN
 F 2 "" H 5300 5700 50  0001 C CNN
@@
 Connection ~ 5500 5500
 $Comp
-L power:GND #PWR?
+L power:GND #PWR0104
 U 1 1 5B9F4DB8
 P 2650 4650
-F 0 "#PWR?" H 2650 4400 50  0001 C CNN
+F 0 "#PWR0104" H 2650 4400 50  0001 C CNN
 F 1 "GND" H 2655 4477 50  0000 C CNN
 F 2 "" H 2650 4650 50  0001 C CNN
@@
 	2950 4500 3250 4500
 $Comp
-L Sensor_Temperature:BD1020HFV U?
+L Sensor_Temperature:BD1020HFV U1
 U 1 1 5B9F57E0
 P 2100 3100
-F 0 "U?" H 2100 3467 50  0000 C CNN
+F 0 "U1" H 2100 3467 50  0000 C CNN
 F 1 "BD1020HFV" H 2100 3376 50  0000 C CNN
 F 2 "Package_TO_SOT_SMD:HVSOF5" H 2100 2700 50  0001 C CNN
@@
 	1550 2700 1550 3000
 $Comp
-L power:GND #PWR?
+L power:GND #PWR0105
 U 1 1 5B9F6328
 P 2500 3350
-F 0 "#PWR?" H 2500 3100 50  0001 C CNN
+F 0 "#PWR0105" H 2500 3100 50  0001 C CNN
 F 1 "GND" H 2505 3177 50  0000 C CNN
 F 2 "" H 2500 3350 50  0001 C CNN
@@
 REMEMBER TO CHECK ALL MAXIMUM VOLTAGE RATINGS\n
 $Comp
-L Connector:USB_B_Micro J?
+L Connector:USB_B_Micro J1
 U 1 1 5B9F7E9F
 P 2650 5500
-F 0 "J?" H 2705 5967 50  0000 C CNN
+F 0 "J1" H 2705 5967 50  0000 C CNN
 F 1 "USB_B_Micro" H 2705 5876 50  0000 C CNN
 F 2 "" H 2800 5450 50  0001 C CNN
@@
 	3250 5500 3250 4700
 $Comp
-L Device:LED D?
+L Device:LED D1
 U 1 1 5B9F95F6
 P 1450 6400
-F 0 "D?" V 1488 6283 50  0000 R CNN
+F 0 "D1" V 1488 6283 50  0000 R CNN
 F 1 "LED" V 1397 6283 50  0000 R CNN
 F 2 "" H 1450 6400 50  0001 C CNN
@@
 $EndComp
 $Comp
-L Device:R R?
+L Device:R R1
 U 1 1 5B9FA85A
 P 1100 6000
-F 0 "R?" H 1170 6046 50  0000 L CNN
+F 0 "R1" H 1170 6046 50  0000 L CNN
 F 1 "R" H 1170 5955 50  0000 L CNN
 F 2 "" V 1030 6000 50  0001 C CNN
@@
 $EndComp
 $Comp
-L Device:R R?
+L Device:R R2
 U 1 1 5B9FA95C
 P 1100 6450
-F 0 "R?" H 1170 6496 50  0000 L CNN
+F 0 "R2" H 1170 6496 50  0000 L CNN
 F 1 "R" H 1170 6405 50  0000 L CNN
 F 2 "" V 1030 6450 50  0001 C CNN
@@
 	1100 6150 1100 6250
 $Comp
-L power:GND #PWR?
+L power:GND #PWR0106
 U 1 1 5B9FBDFD
 P 1100 6850
-F 0 "#PWR?" H 1100 6600 50  0001 C CNN
+F 0 "#PWR0106" H 1100 6600 50  0001 C CNN
 F 1 "GND" H 1105 6677 50  0000 C CNN
 F 2 "" H 1100 6850 50  0001 C CNN
@@
 	7300 2600 7300 2750
 $Comp
-L Switch:SW_Push_Open SW?
+L Switch:SW_Push_Open SW1
 U 1 1 5B9FE51E
 P 7400 2400
-F 0 "SW?" V 7354 2477 50  0000 L CNN
+F 0 "SW1" V 7354 2477 50  0000 L CNN
 F 1 "SW_Push_Open" V 7445 2477 50  0000 L CNN
 F 2 "" H 7400 2600 50  0001 C CNN
@@
 	6200 1900 6200 2200
 $Comp
-L Custom_Symbols:MS5637 U?
+L Custom_Symbols:MS5637 U2
 U 1 1 5BA062B8
 P 3150 1400
-F 0 "U?" H 3150 1515 50  0000 C CNN
+F 0 "U2" H 3150 1515 50  0000 C CNN
 F 1 "MS5637" H 3150 1424 50  0000 C CNN
 F 2 "barometer custom" H 3150 1400 50  0001 C CNN
@@
 	2550 1850 2750 1850
 $Comp
-L power:GND #PWR?
+L power:GND #PWR0107
 U 1 1 5BA215B2
 P 3850 1850
-F 0 "#PWR?" H 3850 1600 50  0001 C CNN
+F 0 "#PWR0107" H 3850 1600 50  0001 C CNN
 F 1 "GND" H 3855 1677 50  0000 C CNN
 F 2 "" H 3850 1850 50  0001 C CNN
@@
 	3850 1850 3550 1850
 $Comp
-L Mechanical:MountingHole_Pad MH?
+L Mechanical:MountingHole_Pad MH1
 U 1 1 5BA25681
 P 1700 4000
-F 0 "MH?" H 2000 4000 50  0000 R CNN
+F 0 "MH1" H 2000 4000 50  0000 R CNN
 F 1 "PRV" H 2000 4100 50  0000 R CNN
 F 2 "" H 1700 4000 50  0001 C CNN
@@
 $EndComp
 $Comp
-L Mechanical:MountingHole_Pad MH?
+L Mechanical:MountingHole_Pad MH2
 U 1 1 5BA25850
 P 1900 4000
-F 0 "MH?" H 1800 3958 50  0000 R CNN
+F 0 "MH2" H 1800 3958 50  0000 R CNN
 F 1 "PRG" H 1800 4050 50  0000 R CNN
 F 2 "" H 1900 4000 50  0001 C CNN
@@
 	1700 3550 1700 3900
 $Comp
-L Device:R R?
+L Device:R R3
 U 1 1 5BA2875E
 P 2250 3800
-F 0 "R?" H 2320 3846 50  0000 L CNN
+F 0 "R3" H 2320 3846 50  0000 L CNN
 F 1 "R" H 2320 3755 50  0000 L CNN
 F 2 "" V 2180 3800 50  0001 C CNN
@@
 	1900 3800 2100 3800
 $Comp
-L power:GND #PWR?
+L power:GND #PWR0108
 U 1 1 5BA3000B
 P 2500 3850
-F 0 "#PWR?" H 2500 3600 50  0001 C CNN
+F 0 "#PWR0108" H 2500 3600 50  0001 C CNN
 F 1 "GND" H 2505 3677 50  0000 C CNN
 F 2 "" H 2500 3850 50  0001 C CNN
@@
 Connection ~ 4950 5550
 $Comp
-L power:+5V #PWR?
+L power:+5V #PWR0109
 U 1 1 5BA3B6F3
 P 1850 4950
-F 0 "#PWR?" H 1850 4800 50  0001 C CNN
+F 0 "#PWR0109" H 1850 4800 50  0001 C CNN
 F 1 "+5V" H 1865 5123 50  0000 C CNN
 F 2 "" H 1850 4950 50  0001 C CNN
@@
 	4950 5550 5300 5550
 $Comp
-L wifi:ESP-WROOM-02 U?
+L wifi:ESP-WROOM-02 U4
 U 1 1 5BA591CF
 P 8750 3600
-F 0 "U?" H 8775 3665 50  0000 C CNN
+F 0 "U4" H 8775 3665 50  0000 C CNN
 F 1 "ESP-WROOM-02" H 8775 3574 50  0000 C CNN
 F 2 "" H 8750 3600 50  0001 C CNN
@@
 VDD
 $Comp
-L power:GND #PWR?
+L power:GND #PWR0110
 U 1 1 5BA5AE20
 P 7900 4900
-F 0 "#PWR?" H 7900 4650 50  0001 C CNN
+F 0 "#PWR0110" H 7900 4650 50  0001 C CNN
 F 1 "GND" H 7905 4727 50  0000 C CNN
 F 2 "" H 7900 4900 50  0001 C CNN
@@
 $EndComp
 $Comp
-L power:GND #PWR?
+L power:GND #PWR0111
 U 1 1 5BA5C912
 P 9900 4800
-F 0 "#PWR?" H 9900 4550 50  0001 C CNN
+F 0 "#PWR0111" H 9900 4550 50  0001 C CNN
 F 1 "GND" H 9905 4627 50  0000 C CNN
 F 2 "" H 9900 4800 50  0001 C CNN
@@
 $EndComp
 $Comp
-L power:GND #PWR?
+L power:GND #PWR0112
 U 1 1 5BA5E404
 P 9900 3900
-F 0 "#PWR?" H 9900 3650 50  0001 C CNN
+F 0 "#PWR0112" H 9900 3650 50  0001 C CNN
 F 1 "GND" H 9905 3727 50  0000 C CNN
 F 2 "" H 9900 3900 50  0001 C CNN
